File: kicad/Project Helena.kicad_pcb (KiCad board)
At the start: 2 copper layers, 346 x 111 mm, 68 parts, among them J1 Conn_01x24, J2 Conn_01x08, J3 Conn_01x08, SW1 BREAK, SW10 H, SW11 SPACE, SW12 HELP, SW13 8, SW14 5, SW15 I, SW16 T, SW17 K, SW18 G, SW19 M, SW2 CONTROL, SW20 B, SW21 START, SW22 9, SW23 4, SW24 O, SW25 R, SW26 L, SW27 F, SW28 COMMA, SW29 V, SW3 SHIFT_L, SW30 SELECT, SW31 0, SW32 3, SW33 P, SW34 E, SW35 SEMICOLON, SW36 D, SW37 PERIOD, SW38 C, SW39 OPTION, SW4 7, SW40 <, SW41 2, SW42 MINUS, SW43 W, SW44 PLUS, SW45 S, SW46 SLASH, SW47 X, SW48 RESET, SW49 >, SW5 6, SW50 1, SW51 EQUAL, SW52 Q, SW53 ASTERISK, SW54 A, SW55 INV, SW56 Z, SW57 DEL, SW58 ESC, SW59 RETURN, SW6 U, SW60 TAB, SW61 CAPS, SW62 SPACE, SW63 SPACE, SW64 SHIFT_R, SW7 Y, SW8 N, SW9 J

Commit message: update silkscreen!
Parts:
- J1: footprint Connector_PinSocket_2.54mm:PinSocket_1x24_P2.54mm_Vertical -> Connector_PinHeader_2.54mm:PinHeader_1x24_P2.54mm_Vertical

Commit message: update of PCB and raytraced image
Other:
- board text added: "ATARI XL KEYBOARD REPLACEMENT"
- board text added: "April 2021 by Ivo van Poorten"
- board text added: "PROJECT HELENA"
- board text added: "REV A"
Changed lines of the file:
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@@
   (general
     (thickness 1.6)
-    (drawings 36)
+    (drawings 41)
     (tracks 437)
     (zones 0)
@@
     (39 F.Mask user)
     (40 Dwgs.User user hide)
-    (41 Cmts.User user hide)
+    (41 Cmts.User user)
     (42 Eco1.User user hide)
     (43 Eco2.User user hide)
@@
     )
   )
+  (dimension 346 (width 0.3) (layer Cmts.User)
+    (gr_text "346.000 mm" (at 203 197.1) (layer Cmts.User)
+      (effects (font (size 1.5 1.5) (thickness 0.3)))
+    )
+    (feature1 (pts (xy 376 189) (xy 376 195.586421)))
+    (feature2 (pts (xy 30 189) (xy 30 195.586421)))
+    (crossbar (pts (xy 30 195) (xy 376 195)))
+    (arrow1a (pts (xy 376 195) (xy 374.873496 195.586421)))
+    (arrow1b (pts (xy 376 195) (xy 374.873496 194.413579)))
+    (arrow2a (pts (xy 30 195) (xy 31.126504 195.586421)))
+    (arrow2b (pts (xy 30 195) (xy 31.126504 194.413579)))
+  )
+  (gr_text "REV A" (at 281.94 162.56) (layer F.SilkS)
+    (effects (font (size 3 3) (thickness 0.6)))
+  )
+  (gr_text "April 2021 by Ivo van Poorten" (at 57.15 165.1) (layer F.SilkS)
+    (effects (font (size 1.5 1.5) (thickness 0.3) italic))
+  )
+  (gr_text "ATARI XL KEYBOARD REPLACEMENT" (at 57.15 162.56) (layer F.SilkS)
+    (effects (font (size 1.5 1.5) (thickness 0.3) italic))
+  )
+  (gr_text "PROJECT HELENA" (at 57.15 158.75) (layer F.SilkS)
+    (effects (font (size 3 3) (thickness 0.6)))
+  )
   (gr_line (start 337 67) (end 337 81) (layer Edge.Cuts) (width 0.15))
